File: source/hub/hub.kicad_sch (KiCad schematic)
At the start: 18 parts, among them J1 10.0 180° ZCJB-HJ, J2 10.0 180° ZCJB-HJ, J3 918-118A2021Y40002, J4 TYPEC-303-ACP16, U1 SL2.1A, X1 12 MHz

Commit message: finished redesigning
Parts:
- X1: footprint Crystal:Crystal_SMD_HC49-SD_HandSoldering -> Crystal:Crystal_SMD_HC49-SD
- renumbered J2 to J1, J3 to J2, J1 to J3
Connections:
- net DM1: now also J1.2 (D-); no longer J3.2 (D-)
- net DM2: now also J3.2 (D-); no longer J1.2 (D-)
- net DP1: now also J1.3 (D+); no longer J3.3 (D+)
- net DP2: now also J3.3 (D+); no longer J1.3 (D+)
Changed lines of the file:
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@@
 		)
 	)
-	(hierarchical_label "DP1"
+	(hierarchical_label "DM1"
 		(shape bidirectional)
-		(at 29.21 22.86 0)
+		(at 27.94 54.61 0)
 		(effects
 			(font
@@
 		)
 	)
-	(hierarchical_label "DP"
+	(hierarchical_label "DP3"
 		(shape bidirectional)
-		(at 123.19 58.42 180)
+		(at 24.13 109.22 180)
 		(effects
 			(font
@@
 		)
 	)
-	(hierarchical_label "DM"
+	(hierarchical_label "DP"
 		(shape bidirectional)
-		(at 123.19 60.96 180)
+		(at 123.19 58.42 180)
 		(effects
 			(font
@@
 		)
 	)
-	(hierarchical_label "DP"
+	(hierarchical_label "DM"
 		(shape bidirectional)
-		(at 123.19 38.1 180)
+		(at 123.19 60.96 180)
 		(effects
 			(font
@@
 		)
 	)
-	(hierarchical_label "DP2"
+	(hierarchical_label "DP"
 		(shape bidirectional)
-		(at 27.94 57.15 0)
+		(at 123.19 38.1 180)
 		(effects
 			(font
 				(size 1.27 1.27)
 			)
-			(justify left)
+			(justify right)
 		)
 	)
 	(hierarchical_label "DP3"
 		(shape bidirectional)
-		(at 46.99 106.68 0)
+		(at 147.32 111.76 0)
 		(effects
 			(font
@@
 		)
 	)
-	(hierarchical_label "DP3"
+	(hierarchical_label "DP1"
 		(shape bidirectional)
-		(at 147.32 111.76 0)
+		(at 27.94 57.15 0)
 		(effects
 			(font
@@
 	(hierarchical_label "DM3"
 		(shape bidirectional)
-		(at 46.99 109.22 0)
+		(at 24.13 106.68 180)
 		(effects
 			(font
 				(size 1.27 1.27)
 			)
-			(justify left)
+			(justify right)
 		)
 	)
-	(hierarchical_label "DP3"
+	(hierarchical_label "DM1"
 		(shape bidirectional)
-		(at 24.13 109.22 180)
+		(at 147.32 104.14 0)
 		(effects
 			(font
 				(size 1.27 1.27)
 			)
-			(justify right)
+			(justify left)
 		)
 	)
-	(hierarchical_label "DM2"
+	(hierarchical_label "DP3"
 		(shape bidirectional)
-		(at 27.94 54.61 0)
+		(at 46.99 106.68 0)
 		(effects
 			(font
@@
 		)
 	)
-	(hierarchical_label "DM1"
+	(hierarchical_label "DM2"
 		(shape bidirectional)
-		(at 147.32 104.14 0)
+		(at 147.32 109.22 0)
 		(effects
 			(font
@@
 		)
 	)
-	(hierarchical_label "DM1"
+	(hierarchical_label "DM3"
 		(shape bidirectional)
-		(at 29.21 20.32 0)
+		(at 46.99 109.22 0)
 		(effects
 			(font
@@
 		)
 	)
-	(hierarchical_label "DM2"
+	(hierarchical_label "DM"
 		(shape bidirectional)
-		(at 147.32 109.22 0)
+		(at 116.84 101.6 180)
 		(effects
 			(font
 				(size 1.27 1.27)
 			)
-			(justify left)
+			(justify right)
 		)
 	)
-	(hierarchical_label "DM3"
+	(hierarchical_label "DM"
 		(shape bidirectional)
-		(at 24.13 106.68 180)
+		(at 123.19 40.64 180)
 		(effects
 			(font
@@
 		)
 	)
-	(hierarchical_label "DM"
+	(hierarchical_label "DM2"
 		(shape bidirectional)
-		(at 116.84 101.6 180)
+		(at 29.21 20.32 0)
 		(effects
 			(font
 				(size 1.27 1.27)
 			)
-			(justify right)
+			(justify left)
 		)
 	)
-	(hierarchical_label "DM"
+	(hierarchical_label "DP1"
 		(shape bidirectional)
-		(at 123.19 40.64 180)
+		(at 147.32 101.6 0)
 		(effects
 			(font
 				(size 1.27 1.27)
 			)
-			(justify right)
+			(justify left)
 		)
 	)
-	(hierarchical_label "DP1"
+	(hierarchical_label "DP2"
 		(shape bidirectional)
-		(at 147.32 101.6 0)
+		(at 29.21 22.86 0)
 		(effects
 			(font
@@
 		(on_board yes)
 		(dnp no)
-		(property "Reference" "J2"
+		(property "Reference" "J1"
 			(at 10.16 48.514 0)
 			(effects
@@
 			(project "hub"
 				(path "/1b2f6184-99b0-41f8-8df3-d5b4aa273ab2"
-					(reference "J2")
+					(reference "J1")
 					(unit 1)
 				)
@@
 		(on_board yes)
 		(dnp no)
-		(property "Reference" "J3"
+		(property "Reference" "J2"
 			(at 26.67 94.996 0)
 			(effects
@@
 			(project "hub"
 				(path "/1b2f6184-99b0-41f8-8df3-d5b4aa273ab2"
-					(reference "J3")
+					(reference "J2")
 					(unit 1)
 				)
@@
 			)
 		)
-		(property "Footprint" "Crystal:Crystal_SMD_HC49-SD_HandSoldering"
+		(property "Footprint" "Crystal:Crystal_SMD_HC49-SD"
 			(at 113.03 120.65 0)
 			(effects
@@
 		(on_board yes)
 		(dnp no)
-		(property "Reference" "J1"
+		(property "Reference" "J3"
 			(at 11.43 14.224 0)
 			(effects
@@
 			(project "hub"
 				(path "/1b2f6184-99b0-41f8-8df3-d5b4aa273ab2"
-					(reference "J1")
+					(reference "J3")
 					(unit 1)
 				)

Commit message: updated missing routes
Connections:
- net +5V: now also C7.1, C8.1, J2.10 (V), J2.15 (V), J2.2 (V), J2.7 (V)
Changed lines of the file:
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@@
+	)
+	(junction
+		(at 17.78 101.6)
+		(diameter 0)
+		(color 0 0 0 0)
 	)
 	(junction
@@
 					(unit 1)
 				)
+			)
+		)
+	)
+	(symbol
+		(lib_id "power:+5V")
+		(at 17.78 101.6 0)
+		(unit 1)
+		(exclude_from_sim no)
+		(in_bom yes)
+		(on_board yes)
+		(dnp no)
+		(property "Reference" "#PWR05"
+			(at 17.78 105.41 0)
+			(effects
+				(font
+					(size 1.27 1.27)
+				)
+				(hide yes)
+			)
+		)
+		(property "Value" "+5V"
+			(at 17.78 96.52 0)
+			(effects
+				(font
+					(size 1.27 1.27)
+				)
+			)
+		)
+		(property "Footprint" ""
+			(at 17.78 101.6 0)
+			(effects
+				(font
+					(size 1.27 1.27)
+				)
+				(hide yes)
+			)
+		)
+		(property "Datasheet" ""
+			(at 17.78 101.6 0)
+			(effects
+				(font
+					(size 1.27 1.27)
+				)
+				(hide yes)
+			)
+		)
+		(property "Description" "Power symbol creates a global label with name \"+5V\""
+			(at 17.78 101.6 0)
+			(effects
+				(font
+					(size 1.27 1.27)
+				)
+				(hide yes)
+			)
+		)
+		(pin "1"
+		)
+		(instances
+			(project "hub"
+				(path "/1b2f6184-99b0-41f8-8df3-d5b4aa273ab2"
+					(reference "#PWR05")
+					(unit 1)
+				)
